File: IRIS-power/5V_supply.sch (KiCad schematic (older format))
At the start: 8 parts, among them U51 TPSM53604

Commit message: Updated to V4.01
Parts:
- C53, C54: Digikey PN (none) -> 1276-3063-1-ND
- R52: Digikey PN RNCP0603FTD2K49CT-ND -> RR08P2.49KDCT-ND
- U51: value TPSM53604 -> TPSM53602; Digikey PN (none) -> 296-TPSM53602RDARDKR-ND
Connections:
- net GND: now also U51.6 (PGOOD)
- no-connect marks 2 -> 1
Other:
- note removed: "Note 1"
- moved on the sheet: C51, C52
Changed lines of the file:
@@
 AR Path="/5F41B5C3/5F427B86" Ref="U51"  Part="1"
 F 0 "U51" H 5700 4400 50  0000 C CNN
-F 1 "TPSM53604" H 5700 4300 50  0000 C CNN
+F 1 "TPSM53602" H 5700 4300 50  0000 C CNN
 F 2 "star-common-lib:TPSM53604" H 5700 3950 50  0001 C CNN
 F 3 "" H 5700 3950 50  0001 C CNN
+F 4 "296-TPSM53602RDARDKR-ND" H 5700 3950 50  0001 C CNN "Digikey PN"
 	1    5700 3950
 	1    0    0    -1
@@
 L Device:C C?
 U 1 1 5F427BA2
-P 4800 3900
+P 4650 3900
 AR Path="/5F427BA2" Ref="C?"  Part="1"
 AR Path="/5F41B5C3/5F427BA2" Ref="C52"  Part="1"
-F 0 "C52" H 4915 3946 50  0000 L CNN
-F 1 "10uF" H 4915 3855 50  0000 L CNN
-F 2 "Capacitor_SMD:C_0603_1608Metric" H 4838 3750 50  0001 C CNN
-F 3 "~" H 4800 3900 50  0001 C CNN
-F 4 "1276-1192-1-ND" H 4800 3900 50  0001 C CNN "Digikey PN"
-	1    4800 3900
+F 0 "C52" H 4765 3946 50  0000 L CNN
+F 1 "10uF" H 4765 3855 50  0000 L CNN
+F 2 "Capacitor_SMD:C_0603_1608Metric" H 4688 3750 50  0001 C CNN
+F 3 "~" H 4650 3900 50  0001 C CNN
+F 4 "1276-1192-1-ND" H 4650 3900 50  0001 C CNN "Digikey PN"
+	1    4650 3900
 	1    0    0    -1
 $EndComp
@@
 L Device:C C?
 U 1 1 5F427BA8
-P 4400 3900
+P 4250 3900
 AR Path="/5F427BA8" Ref="C?"  Part="1"
 AR Path="/5F41B5C3/5F427BA8" Ref="C51"  Part="1"
-F 0 "C51" H 4515 3946 50  0000 L CNN
-F 1 "10uF" H 4515 3855 50  0000 L CNN
-F 2 "Capacitor_SMD:C_0603_1608Metric" H 4438 3750 50  0001 C CNN
-F 3 "~" H 4400 3900 50  0001 C CNN
-F 4 "1276-1192-1-ND" H 4400 3900 50  0001 C CNN "Digikey PN"
-	1    4400 3900
-	1    0    0    -1
-$EndComp
-Wire Wire Line
-	5150 3750 4800 3750
-Connection ~ 5150 3750
-Connection ~ 4800 3750
-Wire Wire Line
-	4800 3750 4400 3750
+F 0 "C51" H 4365 3946 50  0000 L CNN
+F 1 "10uF" H 4365 3855 50  0000 L CNN
+F 2 "Capacitor_SMD:C_0603_1608Metric" H 4288 3750 50  0001 C CNN
+F 3 "~" H 4250 3900 50  0001 C CNN
+F 4 "1276-1192-1-ND" H 4250 3900 50  0001 C CNN "Digikey PN"
+	1    4250 3900
+	1    0    0    -1
+$EndComp
+Connection ~ 4650 3750
+Wire Wire Line
+	4650 3750 4250 3750
 $Comp
 L Device:R R?
@@
 F 2 "Resistor_SMD:R_0603_1608Metric" V 6480 4200 50  0001 C CNN
 F 3 "~" H 6550 4200 50  0001 C CNN
-F 4 "RNCP0603FTD2K49CT-ND" H 6550 4200 50  0001 C CNN "Digikey PN"
+F 4 "RR08P2.49KDCT-ND" H 6550 4200 50  0001 C CNN "Digikey PN"
 	1    6550 4200
 	1    0    0    -1
@@
 L power:GND #PWR?
 U 1 1 5F427BCD
-P 4600 4050
+P 4450 4050
 AR Path="/5F427BCD" Ref="#PWR?"  Part="1"
 AR Path="/5F41B5C3/5F427BCD" Ref="#PWR051"  Part="1"
-F 0 "#PWR051" H 4600 3800 50  0001 C CNN
-F 1 "GND" H 4605 3877 50  0000 C CNN
-F 2 "" H 4600 4050 50  0001 C CNN
-F 3 "" H 4600 4050 50  0001 C CNN
-	1    4600 4050
-	1    0    0    -1
-$EndComp
-Wire Wire Line
-	4400 4050 4600 4050
-Connection ~ 4600 4050
-Wire Wire Line
-	4600 4050 4800 4050
+F 0 "#PWR051" H 4450 3800 50  0001 C CNN
+F 1 "GND" H 4455 3877 50  0000 C CNN
+F 2 "" H 4450 4050 50  0001 C CNN
+F 3 "" H 4450 4050 50  0001 C CNN
+	1    4450 4050
+	1    0    0    -1
+$EndComp
+Wire Wire Line
+	4250 4050 4450 4050
+Connection ~ 4450 4050
+Wire Wire Line
+	4450 4050 4650 4050
 $Comp
 L power:GND #PWR?
@@
 	6550 4400 6550 4350
 Connection ~ 6550 3750
-NoConn ~ 6250 4150
 Wire Wire Line
 	6250 4050 6550 4050
-Text Notes 6600 4100 0    50   ~ 0
-Note 1
-Text HLabel 4400 3750 1    50   Input ~ 0
+Text HLabel 4250 3750 1    50   Input ~ 0
 +BATT
 Text HLabel 8250 3750 2    50   Output ~ 0
@@
 F 2 "Capacitor_SMD:C_1206_3216Metric" H 6988 3750 50  0001 C CNN
 F 3 "~" H 6950 3900 50  0001 C CNN
+F 4 "1276-3063-1-ND" H 6950 3900 50  0001 C CNN "Digikey PN"
 	1    6950 3900
 	1    0    0    -1
@@
 F 2 "Capacitor_SMD:C_1206_3216Metric" H 7588 3750 50  0001 C CNN
 F 3 "~" H 7550 3900 50  0001 C CNN
+F 4 "1276-3063-1-ND" H 7550 3900 50  0001 C CNN "Digikey PN"
 	1    7550 3900
 	1    0    0    -1
@@
 Wire Wire Line
 	7250 4050 7550 4050
+Wire Wire Line
+	4650 3750 5150 3750
+Connection ~ 5150 3750
+$Comp
+L power:GND #PWR?
+U 1 1 5FAE4EFC
+P 6250 4150
+AR Path="/5FAE4EFC" Ref="#PWR?"  Part="1"
+AR Path="/5F41B5C3/5FAE4EFC" Ref="#PWR0102"  Part="1"
+F 0 "#PWR0102" H 6250 3900 50  0001 C CNN
+F 1 "GND" H 6255 3977 50  0000 C CNN
+F 2 "" H 6250 4150 50  0001 C CNN
+F 3 "" H 6250 4150 50  0001 C CNN
+	1    6250 4150
+	1    0    0    -1
+$EndComp
 $EndSCHEMATC

Commit message: IRIS V4.02
Parts:
- U51: footprint star-common-lib:TPSM53604 -> star-common-lib:TPSM53602
Changed lines of the file:
@@
 F 0 "U51" H 5700 4400 50  0000 C CNN
 F 1 "TPSM53602" H 5700 4300 50  0000 C CNN
-F 2 "star-common-lib:TPSM53604" H 5700 3950 50  0001 C CNN
+F 2 "star-common-lib:TPSM53602" H 5700 3950 50  0001 C CNN
 F 3 "" H 5700 3950 50  0001 C CNN
 F 4 "296-TPSM53602RDARDKR-ND" H 5700 3950 50  0001 C CNN "Digikey PN"
