File: IRIS-power/USB_Conn.sch (KiCad schematic (older format))
At the start: 11 parts, among them J81 USB_C_Receptacle_USB2.0, Q81 STS9P3LLH6, U81 TPD2E2U06, U82 STUSB4500LQTR

Commit message: Updated HV supply
Parts:
- removed Q81: STS9P3LLH6, Package_SO:SOP-8_3.9x4.9mm_P1.27mm, symbol star-common-lib:STS9P3LLH6
- added Q81: SSM3J328R, Package_TO_SOT_SMD:SOT-23, symbol Device:Q_PMOS_GSD
- R83: value 20k -> 1k
Connections:
- net VBUS: now also Q81.2 (S)
- net VUSB: now also Q81.3 (D)
- net at R82.2, R83.1: now also Q81.1 (G)
Other:
- moved on the sheet: R82
Changed lines of the file:
@@
 $EndDescr
-$Comp
-L Connector:USB_C_Receptacle_USB2.0 J?
-U 1 1 5FB88211
-P 3800 3900
-AR Path="/5FB88211" Ref="J?"  Part="1"
-AR Path="/5FB7ED68/5FB88211" Ref="J81"  Part="1"
-F 0 "J81" H 3907 4767 50  0000 C CNN
-F 1 "USB_C_Receptacle_USB2.0" H 3907 4676 50  0000 C CNN
-F 2 "Connector_USB:USB_C_Receptacle_GCT_USB4085" H 3950 3900 50  0001 C CNN
-F 3 "https://www.usb.org/sites/default/files/documents/usb_type-c.zip" H 3950 3900 50  0001 C CNN
-	1    3800 3900
-	1    0    0    -1
-$EndComp
 $Comp
 L star-common-lib:STUSB4500LQTR U?
@@
 L power:GND #PWR?
 U 1 1 5FB8823F
-P 5700 4550
+P 5800 4650
 AR Path="/5FB8823F" Ref="#PWR?"  Part="1"
 AR Path="/5FB7ED68/5FB8823F" Ref="#PWR084"  Part="1"
-F 0 "#PWR084" H 5700 4300 50  0001 C CNN
-F 1 "GND" H 5705 4377 50  0000 C CNN
-F 2 "" H 5700 4550 50  0001 C CNN
-F 3 "" H 5700 4550 50  0001 C CNN
-	1    5700 4550
+F 0 "#PWR084" H 5800 4400 50  0001 C CNN
+F 1 "GND" H 5805 4477 50  0000 C CNN
+F 2 "" H 5800 4650 50  0001 C CNN
+F 3 "" H 5800 4650 50  0001 C CNN
+	1    5800 4650
 	1    0    0    -1
 $EndComp
@@
 Wire Wire Line
 	5800 4450 5800 4550
-Wire Wire Line
-	5800 4550 5700 4550
 Connection ~ 5800 4550
 $Comp
@@
 Wire Wire Line
 	3800 4800 3500 4800
-Connection ~ 3800 4800
 Wire Wire Line
 	4500 4050 4500 3600
@@
 L Device:R R?
 U 1 1 5FB8828D
-P 7800 3000
+P 7850 3000
 AR Path="/5FB8828D" Ref="R?"  Part="1"
 AR Path="/5FB7ED68/5FB8828D" Ref="R82"  Part="1"
-F 0 "R82" H 7870 3046 50  0000 L CNN
-F 1 "100k" H 7870 2955 50  0000 L CNN
-F 2 "Resistor_SMD:R_0603_1608Metric" V 7730 3000 50  0001 C CNN
-F 3 "~" H 7800 3000 50  0001 C CNN
-	1    7800 3000
-	1    0    0    -1
-$EndComp
-Wire Wire Line
-	7800 2850 7550 2850
+F 0 "R82" H 7920 3046 50  0000 L CNN
+F 1 "100k" H 7920 2955 50  0000 L CNN
+F 2 "Resistor_SMD:R_0603_1608Metric" V 7780 3000 50  0001 C CNN
+F 3 "~" H 7850 3000 50  0001 C CNN
+	1    7850 3000
+	1    0    0    -1
+$EndComp
 Connection ~ 7200 2850
 Connection ~ 7550 2850
@@
 AR Path="/5FB7ED68/5FB88299" Ref="R83"  Part="1"
 F 0 "R83" H 8320 3346 50  0000 L CNN
-F 1 "20k" H 8320 3255 50  0000 L CNN
+F 1 "1k" H 8320 3255 50  0000 L CNN
 F 2 "Resistor_SMD:R_0603_1608Metric" V 8180 3300 50  0001 C CNN
 F 3 "~" H 8250 3300 50  0001 C CNN
@@
 	1    0    0    -1
 $EndComp
-Wire Wire Line
-	7800 3150 8250 3150
-Wire Wire Line
-	8050 2850 7800 2850
-Connection ~ 7800 2850
 Wire Wire Line
 	8250 3450 8250 3550
@@
 	1    0    0    -1
 $EndComp
-$Comp
-L star-common-lib:STS9P3LLH6 Q81
-U 1 1 5FB9DB9B
+Text HLabel 8650 2850 2    50   Output ~ 0
+VUSB
+Wire Wire Line
+	8650 2850 8550 2850
+Connection ~ 8550 2850
+Wire Wire Line
+	7550 2850 7850 2850
+Wire Wire Line
+	7850 3150 8250 3150
+Connection ~ 8250 3150
+Connection ~ 7850 2850
+$Comp
+L Device:Q_PMOS_GSD Q81
+U 1 1 5FACAFB1
 P 8250 2950
 F 0 "Q81" V 8592 2950 50  0000 C CNN
-F 1 "STS9P3LLH6" V 8501 2950 50  0000 C CNN
-F 2 "Package_SO:SOP-8_3.9x4.9mm_P1.27mm" H 8450 3050 50  0001 C CNN
-F 3 "https://www.st.com/resource/en/datasheet/sts9p3llh6.pdf" H 8250 2950 50  0001 C CNN
+F 1 "SSM3J328R" V 8501 2950 50  0000 C CNN
+F 2 "Package_TO_SOT_SMD:SOT-23" H 8450 3050 50  0001 C CNN
+F 3 "~" H 8250 2950 50  0001 C CNN
 	1    8250 2950
 	0    1    -1   0
 $EndComp
-Connection ~ 8250 3150
-Text HLabel 8650 2850 2    50   Output ~ 0
-VUSB
-Wire Wire Line
-	8650 2850 8550 2850
-Connection ~ 8550 2850
+Wire Wire Line
+	8050 2850 7850 2850
+$Comp
+L Connector:USB_C_Receptacle_USB2.0 J81
+U 1 1 5FACDB97
+P 3800 3900
+F 0 "J81" H 3907 4767 50  0000 C CNN
+F 1 "USB_C_Receptacle_USB2.0" H 3907 4676 50  0000 C CNN
+F 2 "Connector_USB:USB_C_Receptacle_GCT_USB4085" H 3950 3900 50  0001 C CNN
+F 3 "https://www.usb.org/sites/default/files/documents/usb_type-c.zip" H 3950 3900 50  0001 C CNN
+	1    3800 3900
+	1    0    0    -1
+$EndComp
+Connection ~ 3800 4800
+$Comp
+L power:PWR_FLAG #FLG0103
+U 1 1 5FB06030
+P 4600 2850
+F 0 "#FLG0103" H 4600 2925 50  0001 C CNN
+F 1 "PWR_FLAG" H 4600 3023 50  0000 C CNN
+F 2 "" H 4600 2850 50  0001 C CNN
+F 3 "~" H 4600 2850 50  0001 C CNN
+	1    4600 2850
+	1    0    0    -1
+$EndComp
+Connection ~ 4600 2850
+Wire Wire Line
+	5800 4650 5800 4550
 $EndSCHEMATC

Commit message: Updated to V4.01
Parts:
- added FB81: Ferrite_Bead, Inductor_SMD:L_0603_1608Metric, symbol Device:Ferrite_Bead
- added TP101: VBUS, TestPoint:TestPoint_Keystone_5000-5004_Miniature, symbol Connector:TestPoint_Probe
- C81, C82, C83: Digikey PN (none) -> 1276-1860-1-ND
- J81: footprint Connector_USB:USB_C_Receptacle_GCT_USB4085 -> star-common-lib:USB_C_Receptacle_GCT_USB4085_Fixed; Digikey PN (none) -> 2073-USB4085-GF-ACT-ND
- Q81: Digikey PN (none) -> SSM3J328RLFCT-ND
- R81, R83, R84: Digikey PN (none) -> RMCF0603FT1K00CT-ND
- R82: Digikey PN (none) -> RR08P100KDCT-ND
- U81: Digikey PN (none) -> 296-40695-1-ND
- U82: footprint Package_DFN_QFN:QFN-24-1EP_4x4mm_P0.5mm_EP2.7x2.7mm -> star-common-lib:STUSB4500L; Digikey PN (none) -> 497-STUSB4500LQCT-ND
Connections:
- net GND: no longer J81.S1 (SHIELD)
- net VUSB: now also FB81.1; no longer Q81.3 (D), R84.1
- new net: FB81.2, Q81.3 (D), R84.1, TP101.1
- no-connect marks 12 -> 13
Changed lines of the file:
@@
 F 0 "U82" H 6400 4917 50  0000 C CNN
 F 1 "STUSB4500LQTR" H 6400 4826 50  0000 C CNN
-F 2 "Package_DFN_QFN:QFN-24-1EP_4x4mm_P0.5mm_EP2.7x2.7mm" H 6400 3950 50  0001 C CNN
+F 2 "star-common-lib:STUSB4500L" H 6400 3950 50  0001 C CNN
 F 3 "https://www.st.com/resource/en/datasheet/stusb4500l.pdf" H 6400 3950 50  0001 C CNN
+F 4 "497-STUSB4500LQCT-ND" H 6400 3950 50  0001 C CNN "Digikey PN"
 	1    6400 3950
 	1    0    0    -1
@@
 F 2 "Capacitor_SMD:C_0603_1608Metric" H 5538 3350 50  0001 C CNN
 F 3 "~" H 5500 3500 50  0001 C CNN
+F 4 "1276-1860-1-ND" H 5500 3500 50  0001 C CNN "Digikey PN"
 	1    5500 3500
 	1    0    0    -1
@@
 F 2 "Capacitor_SMD:C_0603_1608Metric" H 5138 3350 50  0001 C CNN
 F 3 "~" H 5100 3500 50  0001 C CNN
+F 4 "1276-1860-1-ND" H 5100 3500 50  0001 C CNN "Digikey PN"
 	1    5100 3500
 	1    0    0    -1
@@
 $EndComp
 Wire Wire Line
-	3800 4800 3500 4800
-Wire Wire Line
 	4500 4050 4500 3600
 Wire Wire Line
@@
 F 2 "Capacitor_SMD:C_0603_1608Metric" H 7238 2850 50  0001 C CNN
 F 3 "~" H 7200 3000 50  0001 C CNN
+F 4 "1276-1860-1-ND" H 7200 3000 50  0001 C CNN "Digikey PN"
 	1    7200 3000
 	1    0    0    -1
@@
 F 2 "Resistor_SMD:R_0603_1608Metric" V 7480 3000 50  0001 C CNN
 F 3 "~" H 7550 3000 50  0001 C CNN
+F 4 "RMCF0603FT1K00CT-ND" H 7550 3000 50  0001 C CNN "Digikey PN"
 	1    7550 3000
 	1    0    0    -1
@@
 F 2 "Resistor_SMD:R_0603_1608Metric" V 7780 3000 50  0001 C CNN
 F 3 "~" H 7850 3000 50  0001 C CNN
+F 4 "RR08P100KDCT-ND" H 7850 3000 50  0001 C CNN "Digikey PN"
 	1    7850 3000
 	1    0    0    -1
@@
 F 2 "Resistor_SMD:R_0603_1608Metric" V 8180 3300 50  0001 C CNN
 F 3 "~" H 8250 3300 50  0001 C CNN
+F 4 "RMCF0603FT1K00CT-ND" H 8250 3300 50  0001 C CNN "Digikey PN"
 	1    8250 3300
 	1    0    0    -1
@@
 F 2 "Resistor_SMD:R_0603_1608Metric" V 8480 3000 50  0001 C CNN
 F 3 "~" H 8550 3000 50  0001 C CNN
+F 4 "RMCF0603FT1K00CT-ND" H 8550 3000 50  0001 C CNN "Digikey PN"
 	1    8550 3000
 	1    0    0    -1
@@
 F 2 "Package_TO_SOT_SMD:SOT-23" H 4100 4250 50  0001 C CNN
 F 3 "http://www.ti.com/lit/ds/symlink/tpd2e2u06.pdf" H 4700 4700 50  0001 C CNN
+F 4 "296-40695-1-ND" H 4900 4500 50  0001 C CNN "Digikey PN"
 	1    4900 4500
 	1    0    0    -1
 $EndComp
-Text HLabel 8650 2850 2    50   Output ~ 0
+Text HLabel 9550 2850 2    50   Output ~ 0
 VUSB
-Wire Wire Line
-	8650 2850 8550 2850
-Connection ~ 8550 2850
 Wire Wire Line
 	7550 2850 7850 2850
@@
 F 2 "Package_TO_SOT_SMD:SOT-23" H 8450 3050 50  0001 C CNN
 F 3 "~" H 8250 2950 50  0001 C CNN
+F 4 "SSM3J328RLFCT-ND" H 8250 2950 50  0001 C CNN "Digikey PN"
 	1    8250 2950
 	0    1    -1   0
@@
 F 0 "J81" H 3907 4767 50  0000 C CNN
 F 1 "USB_C_Receptacle_USB2.0" H 3907 4676 50  0000 C CNN
-F 2 "Connector_USB:USB_C_Receptacle_GCT_USB4085" H 3950 3900 50  0001 C CNN
+F 2 "star-common-lib:USB_C_Receptacle_GCT_USB4085_Fixed" H 3950 3900 50  0001 C CNN
 F 3 "https://www.usb.org/sites/default/files/documents/usb_type-c.zip" H 3950 3900 50  0001 C CNN
+F 4 "2073-USB4085-GF-ACT-ND" H 3800 3900 50  0001 C CNN "Digikey PN"
 	1    3800 3900
 	1    0    0    -1
 $EndComp
-Connection ~ 3800 4800
 $Comp
 L power:PWR_FLAG #FLG0103
@@
 Wire Wire Line
 	5800 4650 5800 4550
+NoConn ~ 3500 4800
+$Comp
+L Device:Ferrite_Bead FB81
+U 1 1 5FD50777
+P 9200 2850
+F 0 "FB81" V 8926 2850 50  0000 C CNN
+F 1 "Ferrite_Bead" V 9017 2850 50  0000 C CNN
+F 2 "Inductor_SMD:L_0603_1608Metric" V 9130 2850 50  0001 C CNN
+F 3 "~" H 9200 2850 50  0001 C CNN
+	1    9200 2850
+	0    1    1    0
+$EndComp
+Connection ~ 8550 2850
+Wire Wire Line
+	9350 2850 9550 2850
+$Comp
+L Connector:TestPoint_Probe TP?
+U 1 1 5FD685E7
+P 8600 2700
+AR Path="/5FD685E7" Ref="TP?"  Part="1"
+AR Path="/5FB7ED68/5FD685E7" Ref="TP101"  Part="1"
+F 0 "TP101" H 8753 2801 50  0000 L CNN
+F 1 "VBUS" H 8753 2710 50  0000 L CNN
+F 2 "TestPoint:TestPoint_Keystone_5000-5004_Miniature" H 8800 2700 50  0001 C CNN
+F 3 "~" H 8800 2700 50  0001 C CNN
+F 4 "36-5006-ND" H 8600 2700 50  0001 C CNN "Digikey PN"
+	1    8600 2700
+	1    0    0    -1
+$EndComp
+Wire Wire Line
+	8550 2850 8550 2700
+Wire Wire Line
+	8550 2700 8600 2700
+Wire Wire Line
+	8550 2850 9050 2850
 $EndSCHEMATC

Commit message: IRIS V4.02
Parts:
- added TP81, TP82: TestPoint_Probe, TestPoint:TestPoint_Pad_D2.0mm, symbol Connector:TestPoint_Probe
- FB81: Digikey PN (none) -> BLM18SG700TN1D
Connections:
- net at U82.14 (RP_1A5): now also TP82.1
- net at U82.20 (RP_3A): now also TP81.1
- no-connect marks 13 -> 11
Changed lines of the file:
@@
 NoConn ~ 7000 4150
 NoConn ~ 7000 4050
-NoConn ~ 7000 3950
-NoConn ~ 7000 3850
 Wire Wire Line
 	7000 2850 7000 3250
@@
 F 2 "Inductor_SMD:L_0603_1608Metric" V 9130 2850 50  0001 C CNN
 F 3 "~" H 9200 2850 50  0001 C CNN
+F 4 "BLM18SG700TN1D" H 9200 2850 50  0001 C CNN "Digikey PN"
 	1    9200 2850
 	0    1    1    0
@@
 Wire Wire Line
 	8550 2850 9050 2850
+$Comp
+L Connector:TestPoint_Probe TP81
+U 1 1 5FEEAC57
+P 7550 4000
+F 0 "TP81" H 7703 4101 50  0000 L CNN
+F 1 "TestPoint_Probe" H 7703 4010 50  0000 L CNN
+F 2 "TestPoint:TestPoint_Pad_D2.0mm" H 7750 4000 50  0001 C CNN
+F 3 "~" H 7750 4000 50  0001 C CNN
+	1    7550 4000
+	1    0    0    -1
+$EndComp
+$Comp
+L Connector:TestPoint_Probe TP82
+U 1 1 5FEEB0ED
+P 7550 4400
+F 0 "TP82" H 7703 4501 50  0000 L CNN
+F 1 "TestPoint_Probe" H 7703 4410 50  0000 L CNN
+F 2 "TestPoint:TestPoint_Pad_D2.0mm" H 7750 4400 50  0001 C CNN
+F 3 "~" H 7750 4400 50  0001 C CNN
+	1    7550 4400
+	1    0    0    -1
+$EndComp
+Wire Wire Line
+	7000 3850 7450 3850
+Wire Wire Line
+	7450 3850 7450 4000
+Wire Wire Line
+	7450 4000 7550 4000
+Wire Wire Line
+	7000 3950 7350 3950
+Wire Wire Line
+	7350 3950 7350 4400
+Wire Wire Line
+	7350 4400 7550 4400
 $EndSCHEMATC
